File: hard/TBOT.kicad_sch (KiCad schematic)
At the start: 47 parts, among them J1 BATTERY, J2 R_POWER, J3 L_POWER, J4 OLED_I2C, J5 RTC_I2C, J6 GP_I2C, Q1 ZXMP3A16G, Q2 FDN340P, SW1 SW_SPDT, SW2 SW_DPDT_x2, U1 TBOT_Motor_Driver_R, U2 TBOT_Motor_Driver_L, U3 INA169, U4 CPR_Encoder_R, U5 CPR_Encoder_L, U6 uA7805, U7 MPU-6050_Module

Commit message: Update with pcb
Parts:
- removed R13: 0R NI, Resistor_SMD:R_0805_2012Metric, symbol Device:R
- removed U1: TBOT_Motor_Driver_R, Connector_PinHeader_2.54mm:PinHeader_1x07_P2.54mm_Vertical, symbol Driver_Motor:TBOT_Motor_Driver
- removed U2: TBOT_Motor_Driver_L, Connector_PinHeader_2.54mm:PinHeader_1x07_P2.54mm_Vertical, symbol Driver_Motor:TBOT_Motor_Driver
- removed U4: CPR_Encoder_R, TerminalBlock:TerminalBlock_bornier-4_P5.08mm, symbol Device:CPR_Encoder
- removed U5: CPR_Encoder_L, TerminalBlock:TerminalBlock_bornier-4_P5.08mm, symbol Device:CPR_Encoder
- removed U7: MPU-6050_Module, Connector_PinSocket_2.54mm:PinSocket_1x08_P2.54mm_Vertical, symbol Sensor_Motion:MPU-6050_Module
- added J10: TBOT_Motor_Driver_R, Connector_PinHeader_2.54mm:PinHeader_1x04_P2.54mm_Vertical, symbol Connector_Generic:Conn_01x04
- added J12: CPR_Encoder_R, TerminalBlock_Phoenix:TerminalBlock_Phoenix_MPT-0,5-4-2.54_1x04_P2.54mm_Horizontal, symbol Connector_Generic:Conn_01x04
- added J2: HC-05 Bluetooth module, Connector_PinSocket_2.54mm:PinSocket_1x04_P2.54mm_Horizontal, symbol Connector_Generic:Conn_01x04
- added J3: (no value), symbol Connector_Generic:Conn_01x04
- added J7: TBOT_Motor_Driver_L, Connector_PinHeader_2.54mm:PinHeader_1x04_P2.54mm_Vertical, symbol Connector_Generic:Conn_01x04
- added J9: CPR_Encoder_L, TerminalBlock_Phoenix:TerminalBlock_Phoenix_MPT-0,5-4-2.54_1x04_P2.54mm_Horizontal, symbol Connector_Generic:Conn_01x04
- added R12: 0R NI, Resistor_SMD:R_0805_2012Metric, symbol Device:R
- C1: renamed from C2; value 100nF/10V -> 100nF/20V
- C2: renamed from C1; value 100nF/10V -> 100nF/20V
- C3: renamed from C4; value 10uF/20V -> 1uF/20V
- C5: renamed from C6; value 0.1uF/10V -> 100nF/20V
- C6: renamed from C3; value 100nF/10V -> 100nF/20V
- C8: value 100nF/10V -> 100nF/20V
- D1: footprint Diode_SMD:D_0805_2012Metric -> Diode_SMD:D_SOD-323
- D2: value BZX384A10Q -> 10V
- J1: value BATTERY -> (none); footprint TerminalBlock:TerminalBlock_bornier-2_P5.08mm -> (none)
- J11: renamed from J2; value R_POWER -> (none); footprint TerminalBlock:TerminalBlock_bornier-2_P5.08mm -> (none)
- J8: renamed from J3; value L_POWER -> (none); footprint TerminalBlock:TerminalBlock_bornier-2_P5.08mm -> (none)
- Q1: value ZXMP3A16G -> NDT452AP
- R10: renamed from R11; value R -> (none); footprint Resistor_SMD:R_0805_2012Metric -> (none)
- R9: renamed from R10; value 33k -> 68k
- SW1: value SW_SPDT -> (none)
- U2: renamed from U6; value uA7805 -> UA78M05IDCY
- renumbered C5 to C4, R3 to R1, R14 to R11, R15 to R13, R8 to R14, R9 to R15, R4 to R2, R1 to R3, R2 to R4, R12 to R8, U3 to U1
Connections:
- net +12V: no longer C7.1
- net +3V3: now also J2.1 (Pin_1), J3.1 (Pin_1)
- net +5V: now also J12.1 (Pin_1), J9.1 (Pin_1)
- net BLE_RX: now also J2.3 (Pin_3)
- net BLE_TX: now also J2.4 (Pin_4)
- net GND: now also J10.4 (Pin_4), J12.4 (Pin_4), J2.2 (Pin_2), J3.2 (Pin_2), J7.4 (Pin_4), J9.4 (Pin_4)
- net I2C_SCL: now also XA1.SCL, J3.3 (Pin_3); no longer XA1.D21 (D21_SCL)
- net I2C_SDA: now also XA1.SDA, J3.4 (Pin_4); no longer XA1.D20 (D20_SDA)
- net L_ENCODER_A: now also J9.2 (Pin_2)
- net L_ENCODER_B: now also J9.3 (Pin_3), R12.2; no longer XA1.D10
- net L_FORWARD: now also J7.2 (Pin_2)
- net L_REVERSE: now also J7.3 (Pin_3)
- net M_EN: now also J10.1 (Pin_1), J7.1 (Pin_1)
- net RX: now also SW2.1 (A)
- net R_ENCODER_A: now also XA1.D5, J12.2 (Pin_2)
- net R_ENCODER_B: now also J12.3 (Pin_3)
- net R_FORWARD: now also J10.2 (Pin_2)
- net R_REVERSE: now also J10.3 (Pin_3)
- net TX: now also SW2.4 (A)
- net VDD: now reaches R8.2, XA1.VIN
- net VDD: now also C7.1
- net D: now reaches Q1.2 (D), R5.1, SW1.1 (A)
- new net: R12.1, XA1.D10
- no-connect marks 75 -> 63
Other:
- note added: "0 -> 5 A 0 -> 3.4 V"
- note added: "Arduino mega / Arduino Uno / Nucléo 64 Arduino Uno pin compatible"
- note added: "Bluetooth module"
- note added: "Buzzer"
- note added: "Decoupling"
- note added: "INA169"
- note added: "Left motor"
- note added: "MCU"
- note added: "PMOS 5A 30V"
- note added: "Power"
- note added: "Right motor"
- note removed: "0 -> 10 A 0 -> 3.3 V"
- note removed: "Bornier"
- note removed: "Motor driver"
- note removed: "USB_RX"
- note removed: "USB_TX"
- moved on the sheet: BZ1, C1, C2, C3, C4, C5, C6, C7, C8, D1, D2, D3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

Commit message: Add jumper for Bluetooth selection
Parts:
- removed SW2: SW_DPDT_x2, symbol Switch:SW_DPDT_x2
- added JP1: Jumper_4_Open, symbol Jumper:Jumper_4_Open
- J1: value (none) -> BATTERY; footprint (none) -> TerminalBlock_Phoenix:TerminalBlock_Phoenix_MKDS-1,5-2-5.08_1x02_P5.08mm_Horizontal
- J11: value (none) -> R_POWER; footprint (none) -> TerminalBlock_Phoenix:TerminalBlock_Phoenix_MKDS-1,5-2-5.08_1x02_P5.08mm_Horizontal
- J3: value (none) -> MPU-6050_Module; footprint (none) -> Module:MPU-6050_Module
- J8: value (none) -> L_POWER; footprint (none) -> TerminalBlock_Phoenix:TerminalBlock_Phoenix_MKDS-1,5-2-5.08_1x02_P5.08mm_Horizontal
- R10: value (none) -> 1K; footprint (none) -> Resistor_SMD:R_0805_2012Metric
- SW1: value (none) -> SW_SPDT; footprint (none) -> Button_Switch_THT:5638A
- renumbered R8 to R7, R7 to R8
Connections:
- net RX: now also JP1.3 (C)
- net TX: now also JP1.1 (A)
- net BLE_RX renamed BLUETOOTH_TX
- net BLUETOOTH_TX: now also JP1.2 (B)
- net BLE_TX renamed BLUETOOTH_RX
- net BLUETOOTH_RX: now also JP1.4 (D)
- no-connect marks 63 -> 64

Commit message: First version of TBOT hardware
Parts:
- removed Q2: FDN340P, Package_TO_SOT_SMD:SOT-23, symbol Transistor_FET:FDN340P
- added Q2: DMN2050L, Package_TO_SOT_SMD:SOT-23, symbol Transistor_FET:DMN2050L
- JP1: footprint (none) -> Connector_PinHeader_2.54mm:PinHeader_2x02_P2.54mm_Vertical
- R1: value 9.1K -> 0R
- R2: value 3.6K -> 0R NI
- renumbered R7 to R10, R15 to R14, R14 to R15, R8 to R7, R9 to R8, R10 to R9
Connections:
- net +5V: now also BZ1.1 (-), R14.2
- net GND: now also Q2.2 (S); no longer BZ1.2 (+), U2.4 (GND)
- net RX: now also JP1.1 (A); no longer JP1.3 (C)
- net TX: now also JP1.3 (C); no longer JP1.1 (A)
- net at R15.2: now also Q2.1 (G)
- net +3V3 renamed +3.3V
- new net: BZ1.2 (+), Q2.3 (D)
Other:
- note removed: "Change resistor value"
- moved on the sheet: BZ1, R10, R14, R15
